File: pcb/Power-Module/SEPIC-12V.kicad_sch (KiCad schematic)
At the start: 0 parts

Commit message: 12V and 3.3V supplies in correct form factor
Completed layout of 3.3V out buck converter and 12V out SEPIC converter. Layout fits on board with the same shape and hole pattern as the rev 1 Ride-Along Module.
Parts:
- added C10: 100pF, Capacitor_SMD:C_0603_1608Metric_Pad1.08x0.95mm_HandSolder, symbol Device:C
- added C11: 56pF, Capacitor_SMD:C_0603_1608Metric_Pad1.08x0.95mm_HandSolder, symbol Device:C
- added C12: 5.6nF, Capacitor_SMD:C_0603_1608Metric_Pad1.08x0.95mm_HandSolder, symbol Device:C
- added C13: 1uF, Capacitor_SMD:C_0603_1608Metric_Pad1.08x0.95mm_HandSolder, symbol Device:C
- added C14: 68nF, Capacitor_SMD:C_0603_1608Metric_Pad1.08x0.95mm_HandSolder, symbol Device:C
- added C15: 120pF, Capacitor_SMD:C_0603_1608Metric_Pad1.08x0.95mm_HandSolder, symbol Device:C
- added C16: 8.2uF, Capacitor_SMD:C_0603_1608Metric_Pad1.08x0.95mm_HandSolder, symbol Device:C
- added C8: 4.7uF, Capacitor_SMD:C_0603_1608Metric_Pad1.08x0.95mm_HandSolder, symbol Device:C_Small
- added C9: 25SVPF100M, Capacitor_SMD:CP_Elec_8x6.9, symbol Device:C_Polarized_US
- added D1: B560C-13-F, Diode_SMD:D_SMC_Handsoldering, symbol Device:D_Schottky
- added L2: SRF1260-6R8Y, Inductor_SMD:L_Bourns_SRF1260, symbol Device:L_Coupled_1324
- added Q1: CSD18534Q5A, Package_TO_SOT_SMD:TDSON-8-1, symbol Transistor_FET:CSD18534Q5A
- added R3: 11.3, Resistor_SMD:R_0603_1608Metric_Pad0.98x0.95mm_HandSolder, symbol Device:R_US
- added R4: 1k, Resistor_SMD:R_0603_1608Metric_Pad0.98x0.95mm_HandSolder, symbol Device:R_US
- added R5: 12m, Resistor_SMD:R_1206_3216Metric_Pad1.30x1.75mm_HandSolder, symbol Device:R_US
- added R6: 215k, Resistor_SMD:R_0603_1608Metric_Pad0.98x0.95mm_HandSolder, symbol Device:R_US
- added R7: 4.75k, Resistor_SMD:R_0603_1608Metric_Pad0.98x0.95mm_HandSolder, symbol Device:R_US
- added R8: 18.7k, Resistor_SMD:R_0603_1608Metric_Pad0.98x0.95mm_HandSolder, symbol Device:R_US
- added R9: 162k, Resistor_SMD:R_0603_1608Metric_Pad0.98x0.95mm_HandSolder, symbol Device:R_US
- added U2: TPS40211, Package_SO:VSSOP-10_3x3mm_P0.5mm, symbol Rowan-Rocketry:TPS40211
Connections:
- new net: C15.2, R9.2, U2.1 (RC)
- new net: C13.2, U2.9 (BP)
- new net: Q1.4 (G), R3.2
- new net: C8.1, L2.4, Q1.5 (D)
- new net: C8.2, D1.2 (A), L2.3
- new net: C12.1, R8.1
- new net: Q1.1 (S), Q1.2 (S), Q1.3 (S), R4.2, R5.2
- new net: C14.1, U2.2 (SS)
- new net +12V: C9.1, D1.1 (K), R6.2
- new net Comp: C11.2, C12.2, U2.4 (COMP)
- new net Disable: U2.3 (DIS)
- new net Feedback: C11.1, R6.1, R7.2, R8.2, U2.5 (FB)
- new net GND: C10.2, C13.1, C14.2, C15.1, C16.2, C9.2, L2.1, R5.1, R7.1, U2.11 (GND), U2.6 (GND)
- new net Gate Drive: R3.1, U2.8 (GDRV)
- new net I Sense: C10.1, R4.1, U2.7 (ISNS)
- new net VDD: C16.1, L2.2, R9.1, U2.10 (VDD)
Other:
- note added: "9V to 12.6V in to 12V out SEPIC Converter"
- note added: "Compensation"
- note added: "Feedback Divider"
- note added: "Switch Controller"
