File: pcb/Power-Module/_autosave-Power-Module.kicad_sch (KiCad schematic)
At the start: 10 parts, among them J1 Conn_01x02, J2 Conn_01x06_Socket, SW1 SW_DIP_x02

Commit message: 12V and 3.3V supplies in correct form factor
Completed layout of 3.3V out buck converter and 12V out SEPIC converter. Layout fits on board with the same shape and hole pattern as the rev 1 Ride-Along Module.
Parts:
- J2: footprint (none) -> Connector_PinSocket_2.54mm:PinSocket_1x06_P2.54mm_Vertical
Changed lines of the file:
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@@
 			)
 		)
-		(property "Footprint" ""
+		(property "Footprint" "Connector_PinSocket_2.54mm:PinSocket_1x06_P2.54mm_Vertical"
 			(at 134.62 96.52 0)
 			(effects
